Commit message: feat: add sharpa setup and update the retargeting optimal algorithm of markdown doc

File: assets/robots/hands/schunk_hand/schunk_svh_hand_left.urdf (robot description, URDF)
Before this commit: robot svh, 29 links, 28 joints
Joints:
- joint left_hand_j5: mimic joint=left_hand_Thumb_Opposition multiplier=1 offset=0 -> joint=left_hand_Thumb_Opposition multiplier=-1 offset=0
